File: teensy_audio_player_kicad.sch (KiCad schematic (older format))
At the start: 11 parts, among them J1 Conn_02x13_Odd_Even, J2 Conn_01x03_Female, J3 Conn_01x09_Male, Q1 2N3904, U1 Teensy3.6, U2 74LS373, U3 I2S_DAC

Commit message: update PCB for new version with teensy41
Parts:
- removed U1: Teensy3.6, teensy_audio_player_kicad:Teensy35_36, symbol teensy_library:Teensy3.6
- added R4, R5: R-Device, Resistor_THT:R_Axial_DIN0207_L6.3mm_D2.5mm_P10.16mm_Horizontal, symbol teensy_audio_player_kicad-rescue:R-Device
- added U1: Teensy4.1, teensy_audio_player_kicad:Teensy41, symbol teensy_library:Teensy4.1
- C1: symbol Device:CP1 -> teensy_audio_player_kicad-rescue:CP1-Device
- J1: symbol Connector_Generic:Conn_02x13_Odd_Even -> teensy_audio_player_kicad-rescue:Conn_02x13_Odd_Even-Connector_Generic
- J2: symbol Connector:Conn_01x03_Female -> teensy_audio_player_kicad-rescue:Conn_01x03_Female-Connector
- J3: symbol Connector:Conn_01x09_Male -> teensy_audio_player_kicad-rescue:Conn_01x09_Male-Connector
- Q1: symbol Transistor_BJT:2N3904 -> teensy_audio_player_kicad-rescue:2N3904-Transistor_BJT
- R1: footprint Resistor_SMD:R_1206_3216Metric_Pad1.42x1.75mm_HandSolder -> Resistor_THT:R_Axial_DIN0207_L6.3mm_D2.5mm_P10.16mm_Horizontal; symbol Device:R -> teensy_audio_player_kicad-rescue:R-Device
- R2: footprint Resistor_THT:R_Axial_DIN0207_L6.3mm_D2.5mm_P15.24mm_Horizontal -> Resistor_THT:R_Axial_DIN0207_L6.3mm_D2.5mm_P10.16mm_Horizontal; symbol Device:R -> teensy_audio_player_kicad-rescue:R-Device
- R3: symbol Device:R -> teensy_audio_player_kicad-rescue:R-Device
- U2: symbol 74xx:74LS373 -> teensy_audio_player_kicad-rescue:74LS373-74xx
Connections:
- net +3V3: now also R1.1, U1.46 (3V3); no longer R1.2
- net GND: now also R5.2, U1.1 (GND), U1.34 (GND), U1.47 (GND)
- net VCC: now also R4.2, U1.48 (VIN)
- net at U3.5 (BCK): now also U1.43 (21_A7_RX5_BCLK1)
- net CS: now reaches U2.8 (D3)
- net CS: now also U1.12 (10_CS_MQSR)
- net MOSI: now reaches U2.3 (D0)
- net MOSI: now also U1.13 (11_MOSI_CTX1)
- net 24: now reaches J3.2 (Pin_2)
- net 24: now also U1.16 (24_A10_TX6_SCL2)
- net 25: now reaches J3.3 (Pin_3)
- net 25: now also U1.17 (25_A11_RX6_SDA2)
- net 26: now reaches J3.4 (Pin_4)
- net 26: now also U1.18 (26_A12_MOSI1)
- net 27: now reaches J3.6 (Pin_6)
- net 27: now also U1.19 (27_A13_SCK1)
- net 28: now reaches J3.8 (Pin_8)
- net 28: now also U1.20 (28_RX7)
- net 37: now reaches J3.9 (Pin_9)
- net 37: now also U1.29 (37_CS)
- net 38: now reaches J3.7 (Pin_7)
- net 38: now also U1.30 (38_CS1_IN1)
- net 39: now reaches J3.5 (Pin_5)
- net 39: now also U1.31 (39_MISO1_OUT1A)
- net SCK: now reaches U2.7 (D2)
- net SCK: now also U1.35 (13_SCK_LED)
- net RST: now reaches U2.13 (D4)
- net RST: now also U1.36 (14_A0_TX3_SPDIF_OUT)
- net at U3.4 (DIN): now also U1.9 (7_RX2_OUT1A)
- net at U3.3 (LCK): now also U1.42 (20_A6_TX5_LRCLK1)
- net at Q1.3 (C), R3.1: now also U1.7 (5_IN2)
- net CMD_DATA: now reaches U2.4 (D1)
- net CMD_DATA: now also U1.14 (12_MISO_MQSL)
- net at J3.1 (Pin_1): now also R1.2; no longer R1.1
- new net: R4.1, R5.1, U1.44 (22_A8_CTX1)
Other:
- moved on the sheet: R1
